File: hardware/PCB/midi-tel-interface-board/midi-tel-interface-board.kicad_sch (KiCad schematic)
At the start: 17 parts, among them J1 DIN-5_180degree, J2 Conn_01x07_Male, J3 Conn_01x17_Male, J4 Conn_01x03, J5 Conn_01x03, J6 Conn_01x03, J7 Conn_01x03, SW1 SW_Push, U1 Pico

Commit message: update gitignore and pcb files
Parts:
- removed J4, J5, J6, J7: Conn_01x03, Connector_PinHeader_2.54mm:PinHeader_1x03_P2.54mm_Vertical, symbol Connector_Generic:Conn_01x03
- removed RV1, RV3: R_Potentiometer, Potentiometer_THT:Potentiometer_Alps_RK09Y11_Single_Horizontal, symbol Device:R_Potentiometer
- added VR1, VR2: RK09K1110B26, RK09K1110B26:RK09K1110B26, symbol RK09K1110B26:RK09K1110B26
Connections:
- net +3V3: now also VR1.3 (CW), VR2.3 (CW)
- net ADC_mode: now also VR2.2 (WIPER)
- net ADC_pitch: now also VR1.2 (WIPER)
- net GND: now also VR1.1 (CCW), VR2.1 (CCW)

Commit message: fix: put 17 pin connectors for keyboard matrix
Parts:
- J3: footprint Connector_PinHeader_2.54mm:PinHeader_1x13_P2.54mm_Vertical -> Connector_PinHeader_2.54mm:PinHeader_1x17_P2.54mm_Vertical
Other:
- company: (none) -> helixbyte
- title: (none) -> MIDITEL
